File: PCB DESIGN/TESTER - V01/ElectromagnetArray_V01.sch (EAGLE design)
At the start: 44 parts, among them J1 POWER_JACKPTH_LOCK, Q1 IRLB3813, Q2 IRLB3813, Q3 IRLB3813, Q4 IRLB3813

Commit message: Updates to Preliminary Design
Added pull down resistors for the Gate Input on the Transistors.
All opto isolator LEDs are on the 3V3 rail
Parts:
- added R14, R15, R16, R17: 1k, rcl:R-US_0204/7
Connections:
- removed net N$18: Q3.G, R4.2
- new net +3V3: R11.2, R2.2, R6.2, R8.2, U$1.3V3
- new net N$26: Q3.G, R15.2, R4.2
- net GND: now also R14.1, R15.1, R16.1, R17.1
- net N$1: now also R14.2
- net N$24: now also R17.2
- net N$7: now also R16.2
- net V_USB: no longer R11.2, R2.2, R6.2, R8.2
Other:
- moved on the sheet: D3, D5, D6, D8, OK1, OK2, OK3, OK4, R1, R10, R11, R2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
